File: boards/core/sheets/adsr.kicad_sch (KiCad schematic)
At the start: 28 parts, among them U212 4002, U213 LM358, U214 TL072, U215 CD4053B

Commit message: Added schematics docs
Parts:
- renumbered TP206 to TP202
Changed lines of the file:
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@@
 		(on_board yes)
 		(dnp no)
-		(property "Reference" "TP206"
+		(property "Reference" "TP202"
 			(at 172.72 78.105 0)
 			(effects
@@
 		(on_board yes)
 		(dnp no)
-		(property "Reference" "TP206"
+		(property "Reference" "TP202"
 			(at 144.78 90.805 0)
 			(effects
@@
 		(on_board yes)
 		(dnp no)
-		(property "Reference" "TP206"
+		(property "Reference" "TP202"
 			(at 133.35 75.565 0)
 			(effects
@@
 		(on_board yes)
 		(dnp no)
-		(property "Reference" "TP206"
+		(property "Reference" "TP202"
 			(at 214.63 135.255 0)
 			(effects
