File: boards/core/sheets/buffers.kicad_sch (KiCad schematic)
At the start: 7 parts, among them U221 TL072

Commit message: Added schematics docs
Parts:
- renumbered TP206 to TP202, TP206 to TP230
Changed lines of the file:
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@@
 		(on_board yes)
 		(dnp no)
-		(property "Reference" "TP206"
+		(property "Reference" "TP230"
 			(at 157.48 76.835 0)
 			(effects
@@
 		(on_board yes)
 		(dnp no)
-		(property "Reference" "TP206"
+		(property "Reference" "TP202"
 			(at 158.75 123.825 0)
 			(effects
