File: boards/core/sheets/noise-sub.kicad_sch (KiCad schematic)
At the start: 21 parts, among them Q209 BC548C, Q301 MMBT5551, U222 TL072, U228 CD4040BM96

Commit message: Added schematics docs
Parts:
- renumbered TP206 to TP202
Changed lines of the file:
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@@
 		(on_board yes)
 		(dnp no)
-		(property "Reference" "TP206"
+		(property "Reference" "TP202"
 			(at 86.36 65.405 0)
 			(effects
@@
 		(on_board yes)
 		(dnp no)
-		(property "Reference" "TP206"
+		(property "Reference" "TP202"
 			(at 231.14 112.395 0)
 			(effects
