File: boards/core/sheets/output.kicad_sch (KiCad schematic)
At the start: 21 parts, among them U216 NE5532, U217 TL072

Commit message: Added schematics docs
Parts:
- renumbered TP206 to TP202
Changed lines of the file:
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@@
 		(on_board yes)
 		(dnp no)
-		(property "Reference" "TP206"
+		(property "Reference" "TP202"
 			(at 248.92 121.285 0)
 			(effects
@@
 		(on_board yes)
 		(dnp no)
-		(property "Reference" "TP206"
+		(property "Reference" "TP202"
 			(at 64.77 50.165 0)
 			(effects
@@
 		(on_board yes)
 		(dnp no)
-		(property "Reference" "TP206"
+		(property "Reference" "TP202"
 			(at 151.13 38.735 0)
 			(effects
