File: boards/core/sheets/vco1-waveshapers.kicad_sch (KiCad schematic)
At the start: 41 parts, among them U226 TL072, U227 TL072, U6 TL072

Commit message: Added schematics docs
Parts:
- renumbered #R202 to #R201, #RV202 to #RV201, D212 to D203, D213 to D204, TP206 to TP202, U226 to U210, U227 to U211
Changed lines of the file:
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@@
 		(on_board yes)
 		(dnp no)
-		(property "Reference" "TP206"
+		(property "Reference" "TP202"
 			(at 224.79 109.855 0)
 			(effects
@@
 		(dnp no)
 		(fields_autoplaced yes)
-		(property "Reference" "#PWR0353"
+		(property "Reference" "#PWR0269"
 			(at 93.98 162.56 0)
 			(effects
@@
 		(dnp no)
 		(fields_autoplaced yes)
-		(property "Reference" "#PWR0352"
+		(property "Reference" "#PWR0268"
 			(at 87.63 214.63 0)
 			(effects
@@
 		(dnp no)
 		(fields_autoplaced yes)
-		(property "Reference" "#PWR0359"
+		(property "Reference" "#PWR0275"
 			(at 246.38 113.03 0)
 			(effects
@@
 		(dnp no)
 		(fields_autoplaced yes)
-		(property "Reference" "#RV202"
+		(property "Reference" "#RV201"
 			(at 260.35 158.75 0)
 			(effects
@@
 		(dnp no)
 		(fields_autoplaced yes)
-		(property "Reference" "U227"
+		(property "Reference" "U211"
 			(at 105.41 132.08 0)
 			(effects
@@
 		(dnp no)
 		(fields_autoplaced yes)
-		(property "Reference" "#PWR0357"
+		(property "Reference" "#PWR0273"
 			(at 196.85 74.93 0)
 			(effects
@@
 		(dnp no)
 		(fields_autoplaced yes)
-		(property "Reference" "#R202"
+		(property "Reference" "#R201"
 			(at 247.65 153.67 90)
 			(effects
@@
 		(dnp no)
 		(fields_autoplaced yes)
-		(property "Reference" "#PWR0358"
+		(property "Reference" "#PWR0274"
 			(at 242.57 69.85 0)
 			(effects
@@
 		(dnp no)
 		(fields_autoplaced yes)
-		(property "Reference" "#PWR0347"
+		(property "Reference" "#PWR0263"
 			(at 63.5 63.5 0)
 			(effects
@@
 		(dnp no)
 		(fields_autoplaced yes)
-		(property "Reference" "U226"
+		(property "Reference" "U210"
 			(at 31.75 205.74 0)
 			(effects
@@
 		(dnp no)
 		(fields_autoplaced yes)
-		(property "Reference" "#PWR0356"
+		(property "Reference" "#PWR0272"
 			(at 185.42 81.28 0)
 			(effects
@@
 		(on_board yes)
 		(dnp no)
-		(property "Reference" "U227"
+		(property "Reference" "U211"
 			(at 232.41 109.22 0)
 			(effects
@@
 		(dnp no)
 		(fields_autoplaced yes)
-		(property "Reference" "#PWR0355"
+		(property "Reference" "#PWR0271"
 			(at 97.79 64.77 0)
 			(effects
@@
 		(dnp no)
 		(fields_autoplaced yes)
-		(property "Reference" "#PWR0354"
+		(property "Reference" "#PWR0270"
 			(at 95.25 153.67 0)
 			(effects
@@
 		(on_board yes)
 		(dnp no)
-		(property "Reference" "TP206"
+		(property "Reference" "TP202"
 			(at 118.11 150.495 0)
 			(effects
@@
 		(dnp no)
 		(fields_autoplaced yes)
-		(property "Reference" "#PWR0348"
+		(property "Reference" "#PWR0264"
 			(at 64.77 203.2 0)
 			(effects
@@
 		(dnp no)
 		(fields_autoplaced yes)
-		(property "Reference" "U227"
+		(property "Reference" "U211"
 			(at 43.18 205.74 0)
 			(effects
@@
 		(dnp no)
 		(fields_autoplaced yes)
-		(property "Reference" "#PWR0349"
+		(property "Reference" "#PWR0265"
 			(at 64.77 217.17 0)
 			(effects
@@
 		(dnp no)
 		(fields_autoplaced yes)
-		(property "Reference" "D212"
+		(property "Reference" "D203"
 			(at 48.26 123.19 0)
 			(effects
@@
 		(dnp no)
 		(fields_autoplaced yes)
-		(property "Reference" "#PWR0361"
+		(property "Reference" "#PWR0277"
 			(at 257.81 167.64 0)
 			(effects
@@
 		(on_board yes)
 		(dnp no)
-		(property "Reference" "TP206"
+		(property "Reference" "TP202"
 			(at 118.11 61.595 0)
 			(effects
@@
 		(on_board yes)
 		(dnp no)
-		(property "Reference" "TP206"
+		(property "Reference" "TP202"
 			(at 83.82 28.575 0)
 			(effects
@@
 		(dnp no)
 		(fields_autoplaced yes)
-		(property "Reference" "U226"
+		(property "Reference" "U210"
 			(at 212.09 45.72 0)
 			(effects
@@
 		(dnp no)
 		(fields_autoplaced yes)
-		(property "Reference" "#PWR0350"
+		(property "Reference" "#PWR0266"
 			(at 68.58 153.67 0)
 			(effects
@@
 		(dnp no)
 		(fields_autoplaced yes)
-		(property "Reference" "U226"
+		(property "Reference" "U210"
 			(at 252.73 48.26 0)
 			(effects
@@
 		(dnp no)
 		(fields_autoplaced yes)
-		(property "Reference" "#PWR0360"
+		(property "Reference" "#PWR0276"
 			(at 257.81 158.75 0)
 			(effects
@@
 		(dnp no)
 		(fields_autoplaced yes)
-		(property "Reference" "D213"
+		(property "Reference" "D204"
 			(at 48.26 133.35 0)
 			(effects
@@
 		(dnp no)
 		(fields_autoplaced yes)
-		(property "Reference" "#PWR0346"
+		(property "Reference" "#PWR0262"
 			(at 44.45 78.74 0)
 			(effects
@@
 		(on_board yes)
 		(dnp no)
-		(property "Reference" "TP206"
+		(property "Reference" "TP202"
 			(at 266.7 66.675 0)
 			(effects
@@
 		(dnp no)
 		(fields_autoplaced yes)
-		(property "Reference" "#PWR0351"
+		(property "Reference" "#PWR0267"
 			(at 78.74 166.37 0)
 			(effects
@@
 		(dnp no)
 		(fields_autoplaced yes)
-		(property "Reference" "#PWR0345"
+		(property "Reference" "#PWR0261"
 			(at 35.56 69.85 0)
 			(effects
