File: boards/core/experimental/core.kicad_pcb (KiCad board)
At the start: 2 copper layers, 215 x 100 mm, 372 parts, among them J201 Conn_02x08_Counter_Clockwise, J202 Conn_02x08_Counter_Clockwise, J203 Conn_02x08_Counter_Clockwise, J204 Conn_02x08_Counter_Clockwise, J205 Conn_01x03, J206 Conn_01x03, J207 Screw_Terminal_01x03, J208 Conn_01x03, J209 Conn_01x03, J214 Conn_02x04_Counter_Clockwise, Q201 2N3906, Q202 BC847BS, Q203 MMBFJ111, Q204 2N3906, Q205 BC847BS, Q206 MMBFJ111, Q207 BC847BS, Q208 BC548C, Q209 BC548C, Q210 BC548C, Q211 J111, Q212 MMBT5551, Q213 MMBT5551, Q214 MMBT5551, Q215 J111, U201 TL072, U202 TL072, U203 LM311, U204 TL072, U205 TL072, U206 LM311, U207 TL072, U208 TL072, U209 TL072, U210 TL072, U211 TL072, U212 4002, U213 LM358, U214 TL072, U215 CD4053B, U216 NE5532, U217 TL072, U218 TL072, U219 TL072, U220 TL072, U221 TL072, U222 TL072, U223 TL072, U224 LM336M-5.0/TR, U225 TL072, U226 TL072, U227 TL072, U228 CD4040BM96

Commit message: Updated UI board connector positions
https://github.com/shmoergh/hog/issues/31

Moving the tuner trimmers on the Core board required to reposition the connector headers too. This also had to be done on the UI board otherwise it won't be possible to connect the two boards.
Parts:
- removed J208, J209: Conn_01x03, Connector_PinHeader_2.54mm:PinHeader_1x03_P2.54mm_Vertical
- J201, J202, J203, J204: footprint Connector_IDC:IDC-Header_2x08_P2.54mm_Vertical -> Connector_PinHeader_2.54mm:PinHeader_2x08_P2.54mm_Vertical
- J_POWER201: footprint Connector_IDC:IDC-Header_2x05_P2.54mm_Vertical -> Connector_PinHeader_2.54mm:PinHeader_2x05_P2.54mm_Vertical
- moved J206 212.8 mm to (37.0, 181.0)
- moved J_POWER201 204.8 mm to (237.0, 242.0), turned to 0 degrees
- moved J202 7.38 mm to (39.0, 226.0)
- moved J203 0.28 mm to (237.0, 216.0)
- moved J204 0.18 mm to (237.0, 185.0)
- moved J201 0.14 mm to (39.0, 249.0)
Routing:
- net -5V: track 167.5 -> 140.1 mm
- net -12V: track 1088.5 -> 1108.6 mm, vias 25 -> 26
- net /VCO/RAW_SAW: track 190.9 -> 180.9 mm
- net VCO2_AUDIO: track 171.7 -> 174.8 mm
- net VCO1_AUDIO: track 166.4 -> 169.5 mm
- net VCO1_SYNC: track 71.8 -> 68.8 mm
- net VCO2_CV: track 167.4 -> 170.2 mm
- net VCO1_FM: track 86.2 -> 84.3 mm
- net +12V: track 1195.3 -> 1197.2 mm
- net GND: track 234.8 -> 236.6 mm, vias 407 -> 409
- net VCO2_FM: track 136.4 -> 138.1 mm
- net DECAY: track 76.9 -> 78.6 mm
- net RELEASE: track 68.7 -> 70.1 mm
- net VCO1_CV: track 118.1 -> 117.3 mm
- net GLIDED_PITCH: track 110.5 -> 111.1 mm
Other:
- board text added: "12V GND -12V"
- board text removed: "12V"
- board text removed: "5V GND -5V"
