File: boards/core/experimental/core.kicad_sch (KiCad schematic)
At the start: 11 parts, among them J201 Conn_02x08_Counter_Clockwise, J202 Conn_02x08_Counter_Clockwise, J203 Conn_02x08_Counter_Clockwise, J204 Conn_02x08_Counter_Clockwise, J214 Conn_02x04_Counter_Clockwise

Commit message: Updated UI board connector positions
https://github.com/shmoergh/hog/issues/31

Moving the tuner trimmers on the Core board required to reposition the connector headers too. This also had to be done on the UI board otherwise it won't be possible to connect the two boards.
Parts:
- J201, J202, J203, J204: footprint Connector_IDC:IDC-Header_2x08_P2.54mm_Vertical -> Connector_PinHeader_2.54mm:PinHeader_2x08_P2.54mm_Vertical
- J_POWER201: footprint Connector_IDC:IDC-Header_2x05_P2.54mm_Vertical -> Connector_PinHeader_2.54mm:PinHeader_2x05_P2.54mm_Vertical
Changed lines of the file:
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@@
 			)
 		)
-		(property "Footprint" "Connector_IDC:IDC-Header_2x08_P2.54mm_Vertical"
+		(property "Footprint" "Connector_PinHeader_2.54mm:PinHeader_2x08_P2.54mm_Vertical"
 			(at 355.6 46.99 0)
 			(effects
@@
 			)
 		)
-		(property "Footprint" "Connector_IDC:IDC-Header_2x08_P2.54mm_Vertical"
+		(property "Footprint" "Connector_PinHeader_2.54mm:PinHeader_2x08_P2.54mm_Vertical"
 			(at 355.6 78.74 0)
 			(effects
@@
 			)
 		)
-		(property "Footprint" "Connector_IDC:IDC-Header_2x05_P2.54mm_Vertical"
+		(property "Footprint" "Connector_PinHeader_2.54mm:PinHeader_2x05_P2.54mm_Vertical"
 			(at 407.67 110.49 0)
 			(effects
@@
 			)
 		)
-		(property "Footprint" "Connector_IDC:IDC-Header_2x08_P2.54mm_Vertical"
+		(property "Footprint" "Connector_PinHeader_2.54mm:PinHeader_2x08_P2.54mm_Vertical"
 			(at 355.6 114.3 0)
 			(effects
@@
 			)
 		)
-		(property "Footprint" "Connector_IDC:IDC-Header_2x08_P2.54mm_Vertical"
+		(property "Footprint" "Connector_PinHeader_2.54mm:PinHeader_2x08_P2.54mm_Vertical"
 			(at 407.67 46.99 0)
 			(effects
