File: boards/core/experimental/sheets/power.kicad_sch (KiCad schematic)
At the start: 24 parts, among them J202 Screw_Terminal_01x03, J203 Conn_01x03, J204 Conn_01x03, U202 TL072, U204 LM336M-5.0/TR, U223 TL072

Commit message: Updated UI board connector positions
https://github.com/shmoergh/hog/issues/31

Moving the tuner trimmers on the Core board required to reposition the connector headers too. This also had to be done on the UI board otherwise it won't be possible to connect the two boards.
Parts:
- removed J203, J204: Conn_01x03, Connector_PinHeader_2.54mm:PinHeader_1x03_P2.54mm_Vertical, symbol Connector_Generic:Conn_01x03
