File: boards/core/experimental/sheets/vco.kicad_sch (KiCad schematic)
At the start: 54 parts, among them Q201 2N3906, Q202 BC847BS, Q203 MMBFJ111, Q215 J111, Q301 MMBT5551, U201 TL072, U202 TL072, U203 LM311

Commit message: Updated UI board connector positions
https://github.com/shmoergh/hog/issues/31

Moving the tuner trimmers on the Core board required to reposition the connector headers too. This also had to be done on the UI board otherwise it won't be possible to connect the two boards.
Parts:
- renumbered Q215 to Q211
Changed lines of the file:
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@@
 		(on_board yes)
 		(dnp no)
-		(property "Reference" "Q215"
+		(property "Reference" "Q211"
 			(at 222.25 38.354 90)
 			(effects
