File: boards/ui/sheets/adsr-logic.kicad_sch (KiCad schematic)
At the start: 24 parts

Commit message: Removed backpanel IO conn. + fixed drone voltage
https://github.com/shmoergh/hog/issues/37
The IO back panel connector on the UI board is a leftover from an earlier prototype. Can be removed.

https://github.com/shmoergh/hog/issues/36
ATM the gate voltage for drone mode is fixed to 5V which makes it quieter than the normal gate. Drone mode gate voltage should be 8V.
Parts:
- added R48: 47k, Shmoergh_Custom_Footprints:R_Axial_DIN0207_L6.3mm_D2.5mm_P7.62mm_Horizontal, symbol Device:R
- added R49: 100k, Shmoergh_Custom_Footprints:R_Axial_DIN0207_L6.3mm_D2.5mm_P7.62mm_Horizontal, symbol Device:R
Connections:
- net +12V: now also R48.2
- net GND: now also R49.1
- net +5V: no longer names the net of SW_VCO2_WAVE1.4
- net +5V: now also R48.1, R49.2

Commit message: Added production files for the UI board
ref https://github.com/shmoergh/hog/issues/19
Parts:
- C3: Part No. (none) -> 80-C315C474K5R; Part URL (none) -> https://mou.sr/4ggiw21; Vendor (none) -> Mouser
- D2: Part No. (none) -> 625-BZX85C8V2; Part URL (none) -> https://mou.sr/3DeplTn; Vendor (none) -> Mouser
- R2: Part No. (none) -> 603-MFR-25FTF52-200K; Part URL (none) -> https://mou.sr/49BK9jG; Vendor (none) -> Mouser
- R2: Part No. (none) -> 303-MF0W4FF4701A10; Part URL (none) -> https://mou.sr/4fkq2ri; Vendor (none) -> Mouser
- R48: Part No. (none) -> 303-CFR0W4J0473B00; Part URL (none) -> https://mou.sr/49BslVE; Vendor (none) -> Mouser
- R49: Part No. (none) -> 303-MF0W4FF1003T50; Part URL (none) -> https://mou.sr/3BGpE8K; Vendor (none) -> Mouser
- R8: Part No. (none) -> 303-MF0W4FF1002T50; Part URL (none) -> https://mou.sr/3VFoGR5; Vendor (none) -> Mouser
- RV_ATTACK_LONG1, RV_DECAY_SHORT1, RV_RELEASE_MIN3, RV_RELEASE_SHORT1, RV_SUSTAIN_LVL1: Part No. (none) -> 652-3306F-1-104; Part URL (none) -> https://mou.sr/3OVBYFf; Vendor (none) -> Mouser
- RV_ATTACK_SHORT1: Part No. (none) -> 652-3306F-1-103; Part URL (none) -> https://mou.sr/41GreC6; Vendor (none) -> Mouser
- RV_RINGTIME1: Mouser https://hu.mouser.com/ProductDetail/Bourns/PTV112-4420A-A50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 -> (none); Part No. (none) -> 652-PTV1124420AA504; Part URL (none) -> https://mou.sr/47iqFh2; Vendor (none) -> Mouser
- RV_SUSTAIN_MAX1: Part No. (none) -> 652-3306F-1-204; Part URL (none) -> https://mou.sr/3P2IKcd; Vendor (none) -> Mouser
- SW_HOLD1, SW_RING1, SW_SOFT1: Part No. (none) -> TS-22E01AT15; Part URL (none) -> https://www.aliexpress.com/item/32955400123.html?spm=a2g0o.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; Product URL (none) -> https://www.chinadaier.com/6-pin-slide-switch/; Vendor (none) -> Daier
- SW_VCO2_WAVE1: Part No. (none) -> TS23-E02; Part URL (none) -> https://www.aliexpress.com/item/32958319752.html?spm=a2g0o.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; Vendor (none) -> Daier
- TP4, TP5, TP6, TP7, TP_5V1: now left out of the parts list
- U_ADSR_SW_IC1: Part No. (none) -> 595-CD4053BE; Part URL (none) -> https://mou.sr/4a7avII; Vendor (none) -> Mouser

Commit message: Updated resistor Mouser no's and added full bom
- Some of the THT resistors in the BOM were referencing to products with min. 1000 pcs order quantity
- Added a full Mouser BOM which can be used to order all Mouser components by uploading to their BOM tool: https://hu.mouser.com/bom/
Parts:
- R2: Part No. 303-MF0W4FF4701A10 -> 603-MFR-25FBF52-4K7; Part URL https://mou.sr/4fkq2ri -> https://mou.sr/4i8N07f
- R48: Part No. 303-CFR0W4J0473B00 -> 603-MFR-25FTE52-47K; Part URL https://mou.sr/49BslVE -> https://mou.sr/4iUy6Bg
- R49: Part No. 303-MF0W4FF1003T50 -> 603-MFR-25FRF52100K; Part URL https://mou.sr/3BGpE8K -> https://mou.sr/4hEwI4G
- R8: Part No. 303-MF0W4FF1002T50 -> 603-MFR25SFRF52-10K; Part URL https://mou.sr/3VFoGR5 -> https://mou.sr/3XU3MyE
Changed lines of the file:
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@@
 			)
 		)
-		(property "Part No." "303-MF0W4FF1002T50 "
+		(property "Part No." "603-MFR25SFRF52-10K "
 			(at 172.72 81.28 0)
 			(effects
@@
 			)
 		)
-		(property "Part URL" "https://mou.sr/3VFoGR5"
+		(property "Part URL" "https://mou.sr/3XU3MyE"
 			(at 172.72 81.28 0)
 			(effects
@@
 			)
 		)
-		(property "Part No." "303-CFR0W4J0473B00 "
+		(property "Part No." "603-MFR-25FTE52-47K "
 			(at 87.63 144.78 0)
 			(effects
@@
 			)
 		)
-		(property "Part URL" "https://mou.sr/49BslVE"
+		(property "Part URL" "https://mou.sr/4iUy6Bg"
 			(at 87.63 144.78 0)
 			(effects
@@
 			)
 		)
-		(property "Part No." "303-MF0W4FF1003T50 "
+		(property "Part No." "603-MFR-25FRF52100K"
 			(at 87.63 154.94 0)
 			(effects
@@
 			)
 		)
-		(property "Part URL" "https://mou.sr/3BGpE8K"
+		(property "Part URL" "https://mou.sr/4hEwI4G"
 			(at 87.63 154.94 0)
 			(effects
@@
 			)
 		)
-		(property "Part No." "303-MF0W4FF4701A10 "
+		(property "Part No." "603-MFR-25FBF52-4K7"
 			(at 64.77 170.18 0)
 			(effects
@@
 			)
 		)
-		(property "Part URL" "https://mou.sr/4fkq2ri"
+		(property "Part URL" "https://mou.sr/4i8N07f"
 			(at 64.77 170.18 0)
 			(effects
