File: boards/ui/sheets/filter_ui.kicad_sch (KiCad schematic)
At the start: 16 parts

Commit message: Added schematics docs
Parts:
- renumbered RV_RINGTIME1 to RV_RESO_DIRTY1, TP2 to TP27
Changed lines of the file:
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@@
 		(dnp no)
 		(fields_autoplaced yes)
-		(property "Reference" "TP2"
+		(property "Reference" "TP27"
 			(at 111.76 142.748 0)
 			(effects
@@
 		(on_board yes)
 		(dnp no)
-		(property "Reference" "RV_RINGTIME1"
+		(property "Reference" "RV_RESO_DIRTY1"
 			(at 180.34 102.87 0)
 			(effects
@@
 		(on_board yes)
 		(dnp no)
-		(property "Reference" "RV_RINGTIME1"
+		(property "Reference" "RV_RESO_DIRTY1"
 			(at 105.41 157.48 0)
 			(effects

Commit message: Updated RESO pot resistance value
ref. https://github.com/shmoergh/hog/issues/24

UI: Update dirty dual pot to 50kΩ (100kΩ is not available at Mouser)
Parts:
- RV_RESO_DIRTY1: value 100k -> 50k
Changed lines of the file:
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@@
 			)
 		)
-		(property "Value" "100k"
+		(property "Value" "50k"
 			(at 180.34 100.33 0)
 			(effects
@@
 			)
 		)
-		(property "Value" "100k"
+		(property "Value" "50k"
 			(at 105.41 154.94 0)
 			(effects

Commit message: Added production files for the UI board
ref https://github.com/shmoergh/hog/issues/19
Parts:
- J_FILTER_CONN1: Part No. (none) -> 649-1012938191601BLF; Part URL (none) -> https://mou.sr/3ZS3vh3; Vendor (none) -> Mouser
- R9: Part No. (none) -> 303-MF0W4FF1003T50; Part URL (none) -> https://mou.sr/3BGpE8K; Vendor (none) -> Mouser
- R9: Part No. (none) -> 303-MF0W4FF1002T50; Part URL (none) -> https://mou.sr/3VFoGR5; Vendor (none) -> Mouser
- R9: Part No. (none) -> 303-MF0W4FF3303B00; Part URL (none) -> https://mou.sr/3Zu4Yss; Vendor (none) -> Mouser
- RV_ATTACK_LONG1: Part No. (none) -> 652-3306F-1-104; Part URL (none) -> https://mou.sr/3OVBYFf; Vendor (none) -> Mouser
- RV_CUTOFF1: Part No. (none) -> 652-PTV09A4025FB104; Part URL (none) -> https://mou.sr/3Us6dpJ; Vendor (none) -> Mouser
- RV_RESO_DIRTY1: Part No. (none) -> 652-PTV112-4425AB503; Part URL (none) -> https://mou.sr/3UKAAJn; Vendor (none) -> Mouser
- SW_TRACK1: Part No. (none) -> TS-22E01AT15; Part URL (none) -> https://www.aliexpress.com/item/32955400123.html?spm=a2g0o.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; Product URL (none) -> https://www.chinadaier.com/6-pin-slide-switch/; Vendor (none) -> Daier
- TP27: now left out of the parts list

Commit message: Updated resistor Mouser no's and added full bom
- Some of the THT resistors in the BOM were referencing to products with min. 1000 pcs order quantity
- Added a full Mouser BOM which can be used to order all Mouser components by uploading to their BOM tool: https://hu.mouser.com/bom/
Parts:
- R9: Part No. 303-MF0W4FF1003T50 -> 603-MFR-25FRF52100K; Part URL https://mou.sr/3BGpE8K -> https://mou.sr/4hEwI4G
- R9: Part No. 303-MF0W4FF1002T50 -> 603-MFR25SFRF52-10K; Part URL https://mou.sr/3VFoGR5 -> https://mou.sr/3XU3MyE
- R9: Part No. 303-MF0W4FF3303B00 -> 603-MFR-25FRF52-330K; Part URL https://mou.sr/3Zu4Yss -> https://mou.sr/3FzGuYE
Changed lines of the file:
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@@
 		(shape input)
 		(at 130.81 78.74 180)
-		(fields_autoplaced yes)
 		(effects
 			(font
@@
 		(shape input)
 		(at 106.68 46.99 180)
-		(fields_autoplaced yes)
 		(effects
 			(font
@@
 		(shape input)
 		(at 130.81 63.5 180)
-		(fields_autoplaced yes)
 		(effects
 			(font
@@
 			)
 		)
-		(property "Part No." "303-MF0W4FF1003T50 "
+		(property "Part No." "603-MFR-25FRF52100K"
 			(at 137.16 63.5 0)
 			(effects
@@
 			)
 		)
-		(property "Part URL" "https://mou.sr/3BGpE8K"
+		(property "Part URL" "https://mou.sr/4hEwI4G"
 			(at 137.16 63.5 0)
 			(effects
@@
 			)
 		)
-		(property "Part No." "303-MF0W4FF1002T50 "
+		(property "Part No." "603-MFR25SFRF52-10K "
 			(at 137.16 46.99 0)
 			(effects
@@
 			)
 		)
-		(property "Part URL" "https://mou.sr/3VFoGR5"
+		(property "Part URL" "https://mou.sr/3XU3MyE"
 			(at 137.16 46.99 0)
 			(effects
@@
 			)
 		)
-		(property "Part No." "303-MF0W4FF1002T50 "
+		(property "Part No." "603-MFR25SFRF52-10K "
 			(at 142.24 156.21 0)
 			(effects
@@
 			)
 		)
-		(property "Part URL" "https://mou.sr/3VFoGR5"
+		(property "Part URL" "https://mou.sr/3XU3MyE"
 			(at 142.24 156.21 0)
 			(effects
@@
 			)
 		)
-		(property "Part No." "303-MF0W4FF1002T50 "
+		(property "Part No." "603-MFR25SFRF52-10K "
 			(at 142.24 114.3 0)
 			(effects
@@
 			)
 		)
-		(property "Part URL" "https://mou.sr/3VFoGR5"
+		(property "Part URL" "https://mou.sr/3XU3MyE"
 			(at 142.24 114.3 0)
 			(effects
@@
 			)
 		)
-		(property "Part No." "303-MF0W4FF3303B00 "
+		(property "Part No." "603-MFR-25FRF52-330K "
 			(at 137.16 78.74 0)
 			(effects
@@
 			)
 		)
-		(property "Part URL" "https://mou.sr/3Zu4Yss"
+		(property "Part URL" "https://mou.sr/3FzGuYE"
 			(at 137.16 78.74 0)
 			(effects
@@
 			)
 		)
-		(property "Part No." "303-MF0W4FF1003T50 "
+		(property "Part No." "603-MFR-25FRF52100K"
 			(at 137.16 93.98 0)
 			(effects
@@
 			)
 		)
-		(property "Part URL" "https://mou.sr/3BGpE8K"
+		(property "Part URL" "https://mou.sr/4hEwI4G"
 			(at 137.16 93.98 0)
 			(effects
