File: boards/ui/sheets/playground_ui.kicad_sch (KiCad schematic)
At the start: 15 parts

Commit message: Added schematics docs
Parts:
- renumbered TP2 to TP29, TP2 to TP31, TP2 to TP32, TP2 to TP33, TP2 to TP34, TP2 to TP35
Changed lines of the file:
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@@
 		(dnp no)
 		(fields_autoplaced yes)
-		(property "Reference" "TP2"
+		(property "Reference" "TP33"
 			(at 199.39 102.362 0)
 			(effects
@@
 		(dnp no)
 		(fields_autoplaced yes)
-		(property "Reference" "TP2"
+		(property "Reference" "TP31"
 			(at 109.22 57.658 0)
 			(effects
@@
 		(dnp no)
 		(fields_autoplaced yes)
-		(property "Reference" "TP2"
+		(property "Reference" "TP35"
 			(at 139.7 117.602 0)
 			(effects
@@
 		(dnp no)
 		(fields_autoplaced yes)
-		(property "Reference" "TP2"
+		(property "Reference" "TP29"
 			(at 80.01 71.628 0)
 			(effects
@@
 		(dnp no)
 		(fields_autoplaced yes)
-		(property "Reference" "TP2"
+		(property "Reference" "TP32"
 			(at 171.45 62.738 0)
 			(effects
@@
 		(dnp no)
 		(fields_autoplaced yes)
-		(property "Reference" "TP2"
+		(property "Reference" "TP34"
 			(at 213.36 79.248 0)
 			(effects

Commit message: Added production files for the UI board
ref https://github.com/shmoergh/hog/issues/19
Parts:
- C3: Part No. (none) -> 594-K103K15X7RF5TK2; Part URL (none) -> https://mou.sr/49C1dG8; Vendor (none) -> Mouser
- R44, R45: Part No. (none) -> 603-MFR-25FTF52-200K; Part URL (none) -> https://mou.sr/49BK9jG; Vendor (none) -> Mouser
- R50: Part No. (none) -> 303-MF0W4FF1002T50; Part URL (none) -> https://mou.sr/3VFoGR5; Vendor (none) -> Mouser
- RV_ATTACK_LONG1: Part No. (none) -> 652-3306F-1-104; Part URL (none) -> https://mou.sr/3OVBYFf; Vendor (none) -> Mouser
- SW_PLAYGROUND1: Part No. (none) -> 105-SR2512F-34NS; Part URL (none) -> https://mou.sr/3wb0uwA; Vendor (none) -> Mouser
- SW_VCO2_WAVE1: Part No. (none) -> TS23-E02; Part URL (none) -> https://www.aliexpress.com/item/32958319752.html?spm=a2g0o.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; Vendor (none) -> Daier
- TP29, TP31, TP32, TP33, TP34, TP35: now left out of the parts list

Commit message: Updated resistor Mouser no's and added full bom
- Some of the THT resistors in the BOM were referencing to products with min. 1000 pcs order quantity
- Added a full Mouser BOM which can be used to order all Mouser components by uploading to their BOM tool: https://hu.mouser.com/bom/
Parts:
- R50: Part No. 303-MF0W4FF1002T50 -> 603-MFR25SFRF52-10K; Part URL https://mou.sr/3VFoGR5 -> https://mou.sr/3XU3MyE
Changed lines of the file:
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@@
 	(label "PLAYGROUND_DEST"
 		(at 135.89 96.52 0)
-		(fields_autoplaced yes)
 		(effects
 			(font
@@
 	(label "PLAYGROUND_SOURCE"
 		(at 135.89 83.82 0)
-		(fields_autoplaced yes)
 		(effects
 			(font
@@
 		(shape input)
 		(at 102.87 83.82 180)
-		(fields_autoplaced yes)
 		(effects
 			(font
@@
 		(shape output)
 		(at 104.14 104.14 180)
-		(fields_autoplaced yes)
 		(effects
 			(font
@@
 		(shape output)
 		(at 104.14 96.52 180)
-		(fields_autoplaced yes)
 		(effects
 			(font
@@
 		(shape input)
 		(at 102.87 81.28 180)
-		(fields_autoplaced yes)
 		(effects
 			(font
@@
 		(shape input)
 		(at 179.07 102.87 0)
-		(fields_autoplaced yes)
 		(effects
 			(font
@@
 		(shape input)
 		(at 59.69 86.36 180)
-		(fields_autoplaced yes)
 		(effects
 			(font
@@
 			)
 		)
-		(property "Part No." "303-MF0W4FF1002T50 "
+		(property "Part No." "603-MFR25SFRF52-10K "
 			(at 107.95 116.84 0)
 			(effects
@@
 			)
 		)
-		(property "Part URL" "https://mou.sr/3VFoGR5"
+		(property "Part URL" "https://mou.sr/3XU3MyE"
 			(at 107.95 116.84 0)
 			(effects
