File: boards/ui/sheets/vco1_ui.kicad_sch (KiCad schematic)
At the start: 26 parts, among them U1 TL072

Commit message: Added schematics docs
Parts:
- renumbered TP2 to TP10, TP2 to TP11, TP2 to TP12, TP2 to TP13, TP2 to TP14, TP2 to TP15
Changed lines of the file:
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@@
 		(dnp no)
 		(fields_autoplaced yes)
-		(property "Reference" "TP2"
+		(property "Reference" "TP11"
 			(at 129.54 99.568 0)
 			(effects
@@
 		(dnp no)
 		(fields_autoplaced yes)
-		(property "Reference" "TP2"
+		(property "Reference" "TP13"
 			(at 97.79 108.458 0)
 			(effects
@@
 		(dnp no)
 		(fields_autoplaced yes)
-		(property "Reference" "TP2"
+		(property "Reference" "TP10"
 			(at 175.26 90.932 0)
 			(effects
@@
 		(dnp no)
 		(fields_autoplaced yes)
-		(property "Reference" "TP2"
+		(property "Reference" "TP12"
 			(at 128.27 121.412 0)
 			(effects
@@
 		(dnp no)
 		(fields_autoplaced yes)
-		(property "Reference" "TP2"
+		(property "Reference" "TP15"
 			(at 156.21 121.158 0)
 			(effects
@@
 		(dnp no)
 		(fields_autoplaced yes)
-		(property "Reference" "TP2"
+		(property "Reference" "TP14"
 			(at 156.21 103.378 0)
 			(effects

Commit message: Added production files for the UI board
ref https://github.com/shmoergh/hog/issues/19
Parts:
- C3: Part No. (none) -> 594-K103K15X7RF5TK2; Part URL (none) -> https://mou.sr/3VFZIRH; Vendor (none) -> Mouser
- C3: now not fitted; now left out of the parts list
- JP_VCO1_IN1, TP10, TP11, TP12, TP13, TP14, TP15: now left out of the parts list
- R3, R4, R5, R6, R7: value 1.5k (0.1%) -> 10k (0.1%); Part No. (none) -> 660-MF1/4CCT52R1002B; Part URL (none) -> https://mou.sr/4fj3JT3; Vendor (none) -> Mouser
- R8, R9: Part No. (none) -> 303-MF0W4FF1003T50; Part URL (none) -> https://mou.sr/3BGpE8K; Vendor (none) -> Mouser
- R9: Part No. (none) -> 303-MF0W4FF1503B00; Part URL (none) -> https://mou.sr/3BpW47z; Vendor (none) -> Mouser
- RV_ATTACK_LONG1: Part No. (none) -> 652-3306F-1-204; Part URL (none) -> https://mou.sr/3P2IKcd; Vendor (none) -> Mouser
- RV_ATTACK_LONG1: Part No. (none) -> 652-3306F-1-104; Part URL (none) -> https://mou.sr/3OVBYFf; Vendor (none) -> Mouser
- SW_OCTAVE1, SW_WAVESHAPE1: Part No. (none) -> 105-SR2512F-25NS; Part URL (none) -> https://mou.sr/49HHdSv; Vendor (none) -> Mouser
- U1: Part No. (none) -> 595-TL072IP; Part URL (none) -> https://mou.sr/4g5XjI5; Vendor (none) -> Mouser
Other:
- note added: "This jumper is used to be able to tune VCO2 without VCO1."

Commit message: Updated resistor Mouser no's and added full bom
- Some of the THT resistors in the BOM were referencing to products with min. 1000 pcs order quantity
- Added a full Mouser BOM which can be used to order all Mouser components by uploading to their BOM tool: https://hu.mouser.com/bom/
Parts:
- R8, R9: Part No. 303-MF0W4FF1003T50 -> 603-MFR-25FRF52100K; Part URL https://mou.sr/3BGpE8K -> https://mou.sr/4hEwI4G
- R9: Part No. 303-MF0W4FF1503B00 -> 603-MFR-25FBF52-150K; Part URL https://mou.sr/3BpW47z -> https://mou.sr/3DLvBCw
Changed lines of the file:
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@@
 		(shape input)
 		(at 187.96 43.18 180)
-		(fields_autoplaced yes)
 		(effects
 			(font
@@
 		(shape output)
 		(at 180.34 88.9 0)
-		(fields_autoplaced yes)
 		(effects
 			(font
@@
 		(shape input)
 		(at 78.74 127 180)
-		(fields_autoplaced yes)
 		(effects
 			(font
@@
 			)
 		)
-		(property "Part No." "303-MF0W4FF1503B00 "
+		(property "Part No." "603-MFR-25FBF52-150K"
 			(at 121.92 129.54 0)
 			(effects
@@
 			)
 		)
-		(property "Part URL" "https://mou.sr/3BpW47z"
+		(property "Part URL" "https://mou.sr/3DLvBCw"
 			(at 121.92 129.54 0)
 			(effects
@@
 			)
 		)
-		(property "Part No." "303-MF0W4FF1003T50 "
+		(property "Part No." "603-MFR-25FRF52100K"
 			(at 194.31 43.18 0)
 			(effects
@@
 			)
 		)
-		(property "Part URL" "https://mou.sr/3BGpE8K"
+		(property "Part URL" "https://mou.sr/4hEwI4G"
 			(at 194.31 43.18 0)
 			(effects
@@
 			)
 		)
-		(property "Part No." "303-MF0W4FF1003T50 "
+		(property "Part No." "603-MFR-25FRF52100K"
 			(at 194.31 57.15 0)
 			(effects
@@
 			)
 		)
-		(property "Part URL" "https://mou.sr/3BGpE8K"
+		(property "Part URL" "https://mou.sr/4hEwI4G"
 			(at 194.31 57.15 0)
 			(effects
@@
 			)
 		)
-		(property "Part No." "303-MF0W4FF1003T50 "
+		(property "Part No." "603-MFR-25FRF52100K"
 			(at 121.92 140.97 0)
 			(effects
@@
 			)
 		)
-		(property "Part URL" "https://mou.sr/3BGpE8K"
+		(property "Part URL" "https://mou.sr/4hEwI4G"
 			(at 121.92 140.97 0)
 			(effects
@@
 			)
 		)
-		(property "Part No." "303-MF0W4FF1003T50 "
+		(property "Part No." "603-MFR-25FRF52100K"
 			(at 194.31 29.21 0)
 			(effects
@@
 			)
 		)
-		(property "Part URL" "https://mou.sr/3BGpE8K"
+		(property "Part URL" "https://mou.sr/4hEwI4G"
 			(at 194.31 29.21 0)
 			(effects
@@
 			)
 		)
-		(property "Part No." "303-MF0W4FF1003T50 "
+		(property "Part No." "603-MFR-25FRF52100K"
 			(at 194.31 73.66 0)
 			(effects
@@
 			)
 		)
-		(property "Part URL" "https://mou.sr/3BGpE8K"
+		(property "Part URL" "https://mou.sr/4hEwI4G"
 			(at 194.31 73.66 0)
 			(effects
