File: boards/ui/sheets/vco2_ui.kicad_sch (KiCad schematic)
At the start: 33 parts, among them U1 TL072

Commit message: Added schematics docs
Parts:
- renumbered TP2 to TP16, TP2 to TP17, TP2 to TP18, TP2 to TP19, TP2 to TP20, TP2 to TP21, TP2 to TP22, TP2 to TP23, TP2 to TP24
Changed lines of the file:
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@@
 		(dnp no)
 		(fields_autoplaced yes)
-		(property "Reference" "TP2"
+		(property "Reference" "TP18"
 			(at 218.948 93.98 90)
 			(effects
@@
 		(dnp no)
 		(fields_autoplaced yes)
-		(property "Reference" "TP2"
+		(property "Reference" "TP20"
 			(at 137.16 144.272 0)
 			(effects
@@
 		(dnp no)
 		(fields_autoplaced yes)
-		(property "Reference" "TP2"
+		(property "Reference" "TP24"
 			(at 20.32 173.482 0)
 			(effects
@@
 		(dnp no)
 		(fields_autoplaced yes)
-		(property "Reference" "TP2"
+		(property "Reference" "TP19"
 			(at 220.98 123.698 0)
 			(effects
@@
 		(dnp no)
 		(fields_autoplaced yes)
-		(property "Reference" "TP2"
+		(property "Reference" "TP21"
 			(at 24.13 95.758 0)
 			(effects
@@
 		(dnp no)
 		(fields_autoplaced yes)
-		(property "Reference" "TP2"
+		(property "Reference" "TP17"
 			(at 218.948 85.09 90)
 			(effects
@@
 		(dnp no)
 		(fields_autoplaced yes)
-		(property "Reference" "TP2"
+		(property "Reference" "TP16"
 			(at 218.948 76.2 90)
 			(effects
@@
 		(dnp no)
 		(fields_autoplaced yes)
-		(property "Reference" "TP2"
+		(property "Reference" "TP23"
 			(at 24.13 167.132 0)
 			(effects
@@
 		(dnp no)
 		(fields_autoplaced yes)
-		(property "Reference" "TP2"
+		(property "Reference" "TP22"
 			(at 20.32 89.408 0)
 			(effects

Commit message: Added production files for the UI board
ref https://github.com/shmoergh/hog/issues/19
Parts:
- C3: Part No. (none) -> 594-K102M15X7RF53L2; Part URL (none) -> https://mou.sr/3OTl4qX; Vendor (none) -> Mouser
- R10, R9: Part No. (none) -> 303-MF0W4FF1003T50; Part URL (none) -> https://mou.sr/3BGpE8K; Vendor (none) -> Mouser
- R3: Part No. (none) -> 660-MF1/4CCT52R1002B; Part URL (none) -> https://mou.sr/4fj3JT3; Vendor (none) -> Mouser
- R3: Part No. (none) -> 303-MF0W4FF8202B00; Part URL (none) -> https://mou.sr/3Djf3kL; Vendor (none) -> Mouser
- RV1, RV2: Part No. (none) -> 652-3006P-1-503-LF; Part URL (none) -> https://mou.sr/3ZEVzhM; Vendor (none) -> Mouser
- RV_VCO2_TUNER1: Part No. (none) -> 652-PTV09A4025FB104; Part URL (none) -> https://mou.sr/3Us6dpJ; Vendor (none) -> Mouser
- RV_VCO2_VOLUME1: Part No. (none) -> 652-PTV09A-4025UA104; Part URL (none) -> https://mou.sr/44vDepN; Vendor (none) -> Mouser
- SW_VCO2_OCT_AMNT1, SW_VCO2_ON1: Part No. (none) -> TS-22E01AT15; Part URL (none) -> https://www.aliexpress.com/item/32955400123.html?spm=a2g0o.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; Product URL (none) -> https://www.chinadaier.com/6-pin-slide-switch/; Vendor (none) -> Daier
- SW_VCO2_OCT_DIR1, SW_VCO2_WAVE1: Part No. (none) -> TS23-E02; Part URL (none) -> https://www.aliexpress.com/item/32958319752.html?spm=a2g0o.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; Vendor (none) -> Daier
- TP16, TP17, TP18, TP19, TP20, TP21, TP22, TP23, TP24: now left out of the parts list
- U1: Part No. (none) -> 595-TL072IP; Part URL (none) -> https://mou.sr/4g5XjI5; Vendor (none) -> Mouser

Commit message: Updated resistor Mouser no's and added full bom
- Some of the THT resistors in the BOM were referencing to products with min. 1000 pcs order quantity
- Added a full Mouser BOM which can be used to order all Mouser components by uploading to their BOM tool: https://hu.mouser.com/bom/
Parts:
- R10, R9: Part No. 303-MF0W4FF1003T50 -> 603-MFR-25FRF52100K; Part URL https://mou.sr/3BGpE8K -> https://mou.sr/4hEwI4G
- R3: Part No. 303-MF0W4FF8202B00 -> 603-MFR-25FBF52-82K; Part URL https://mou.sr/3Djf3kL -> https://mou.sr/4bFupx1
Changed lines of the file:
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@@
 		(shape output)
 		(at 252.73 53.34 0)
-		(fields_autoplaced yes)
 		(effects
 			(font
@@
 		(shape input)
 		(at 138.43 81.28 180)
-		(fields_autoplaced yes)
 		(effects
 			(font
@@
 		(shape input)
 		(at 138.43 115.57 180)
-		(fields_autoplaced yes)
 		(effects
 			(font
@@
 		(shape input)
 		(at 138.43 38.1 180)
-		(fields_autoplaced yes)
 		(effects
 			(font
@@
 			)
 		)
-		(property "Part No." "303-MF0W4FF1003T50 "
+		(property "Part No." "603-MFR-25FRF52100K"
 			(at 144.78 99.06 0)
 			(effects
@@
 			)
 		)
-		(property "Part URL" "https://mou.sr/3BGpE8K"
+		(property "Part URL" "https://mou.sr/4hEwI4G"
 			(at 144.78 99.06 0)
 			(effects
@@
 			)
 		)
-		(property "Part No." "303-MF0W4FF1003T50 "
+		(property "Part No." "603-MFR-25FRF52100K"
 			(at 229.87 38.1 0)
 			(effects
@@
 			)
 		)
-		(property "Part URL" "https://mou.sr/3BGpE8K"
+		(property "Part URL" "https://mou.sr/4hEwI4G"
 			(at 229.87 38.1 0)
 			(effects
@@
 			)
 		)
-		(property "Part No." "303-MF0W4FF1003T50 "
+		(property "Part No." "603-MFR-25FRF52100K"
 			(at 144.78 134.62 0)
 			(effects
@@
 			)
 		)
-		(property "Part URL" "https://mou.sr/3BGpE8K"
+		(property "Part URL" "https://mou.sr/4hEwI4G"
 			(at 144.78 134.62 0)
 			(effects
@@
 			)
 		)
-		(property "Part No." "303-MF0W4FF1003T50 "
+		(property "Part No." "603-MFR-25FRF52100K"
 			(at 144.78 38.1 0)
 			(effects
@@
 			)
 		)
-		(property "Part URL" "https://mou.sr/3BGpE8K"
+		(property "Part URL" "https://mou.sr/4hEwI4G"
 			(at 144.78 38.1 0)
 			(effects
@@
 			)
 		)
-		(property "Part No." "303-MF0W4FF1003T50 "
+		(property "Part No." "603-MFR-25FRF52100K"
 			(at 144.78 115.57 0)
 			(effects
@@
 			)
 		)
-		(property "Part URL" "https://mou.sr/3BGpE8K"
+		(property "Part URL" "https://mou.sr/4hEwI4G"
 			(at 144.78 115.57 0)
 			(effects
@@
 			)
 		)
-		(property "Part No." "303-MF0W4FF1003T50 "
+		(property "Part No." "603-MFR-25FRF52100K"
 			(at 144.78 81.28 0)
 			(effects
@@
 			)
 		)
-		(property "Part URL" "https://mou.sr/3BGpE8K"
+		(property "Part URL" "https://mou.sr/4hEwI4G"
 			(at 144.78 81.28 0)
 			(effects
@@
 			)
 		)
-		(property "Part No." "303-MF0W4FF8202B00 "
+		(property "Part No." "603-MFR-25FBF52-82K "
 			(at 114.3 54.61 0)
 			(effects
@@
 			)
 		)
-		(property "Part URL" "https://mou.sr/3Djf3kL"
+		(property "Part URL" "https://mou.sr/4bFupx1"
 			(at 114.3 54.61 0)
 			(effects
@@
 			)
 		)
-		(property "Part No." "303-MF0W4FF8202B00 "
+		(property "Part No." "603-MFR-25FBF52-82K "
 			(at 114.3 72.39 0)
 			(effects
@@
 			)
 		)
-		(property "Part URL" "https://mou.sr/3Djf3kL"
+		(property "Part URL" "https://mou.sr/4bFupx1"
 			(at 114.3 72.39 0)
 			(effects
@@
 			)
 		)
-		(property "Part No." "303-MF0W4FF1003T50 "
+		(property "Part No." "603-MFR-25FRF52100K"
 			(at 144.78 50.8 0)
 			(effects
@@
 			)
 		)
-		(property "Part URL" "https://mou.sr/3BGpE8K"
+		(property "Part URL" "https://mou.sr/4hEwI4G"
 			(at 144.78 50.8 0)
 			(effects
@@
 			)
 		)
-		(property "Part No." "303-MF0W4FF1003T50 "
+		(property "Part No." "603-MFR-25FRF52100K"
 			(at 144.78 63.5 0)
 			(effects
@@
 			)
 		)
-		(property "Part URL" "https://mou.sr/3BGpE8K"
+		(property "Part URL" "https://mou.sr/4hEwI4G"
 			(at 144.78 63.5 0)
 			(effects
