File: boards/core/stable/sheets/buffers.kicad_sch (KiCad schematic)
At the start: 7 parts, among them U221 TL072

Commit message: Updated and checked Core board BOM
ref https://github.com/shmoergh/hog/issues/19
Parts:
- C203, C204, R294, R295, U221: Vendor (none) -> JLCPCB
