File: boards/core/stable/sheets/lfos.kicad_sch (KiCad schematic)
At the start: 13 parts, among them Q208 BC548C, U219 TL072

Commit message: Updated and checked Core board BOM
ref https://github.com/shmoergh/hog/issues/19
Parts:
- C203, C204, R201, R288, R290, R292, U219: Vendor (none) -> JLCPCB
- C255: Part No. (none) -> 80-R82EC1330AA50K; Part URL (none) -> https://mou.sr/3BhmOHr; Vendor (none) -> Mouser; now in the parts list
- Q208: Part No. (none) -> 637-BC548C; Part URL (none) -> https://mou.sr/4fhkHkJ; Vendor (none) -> Mouser; now in the parts list
