File: boards/core/stable/sheets/noise-sub.kicad_sch (KiCad schematic)
At the start: 21 parts, among them Q209 BC548C, Q301 MMBT5551, U222 TL072, U228 CD4040BM96

Commit message: Updated and checked Core board BOM
ref https://github.com/shmoergh/hog/issues/19
Parts:
- C208, C209, C220, Q301, R234, R235, R236, R320, R321, R332, R333, R334, R335, R336, R337, U222, U228: Vendor (none) -> JLCPCB
- Q209: Part No. (none) -> 637-BC548C; Part URL (none) -> https://mou.sr/4fhkHkJ; Vendor (none) -> Mouser; now in the parts list
- RV202: value 100k Log -> 100k; Part No. (none) -> 531-PT6KH104A1010PM; Part URL (none) -> https://mou.sr/49zQlIS; Vendor (none) -> Mouser; now in the parts list
