File: boards/core/stable/sheets/power.kicad_sch (KiCad schematic)
At the start: 13 parts, among them J202 Screw_Terminal_01x03, U202 TL072, U223 TL072

Commit message: Streamline 'Stable' Core board
https://github.com/shmoergh/hog/issues/7

- Remove 12V terminal input
- Reposition Eurorack power connector to right so it makes space for tuning
- Remove all unnecessary thermal compensation pseudo components
- Reposition tuning trimmers
Parts:
- removed J202: Screw_Terminal_01x03, TerminalBlock_Phoenix:TerminalBlock_Phoenix_MKDS-1,5-3_1x03_P5.00mm_Horizontal, symbol Connector:Screw_Terminal_01x03
- added J_POWER201: Conn_02x05_Odd_Even, Connector_PinHeader_2.54mm:PinHeader_2x05_P2.54mm_Vertical, symbol Connector_Generic:Conn_02x05_Odd_Even
- added TP235: 12V, TestPoint:TestPoint_THTPad_2.0x2.0mm_Drill1.0mm, symbol Connector:TestPoint
- added TP236: -12V, TestPoint:TestPoint_THTPad_2.0x2.0mm_Drill1.0mm, symbol Connector:TestPoint
- added TP237: -5V, TestPoint:TestPoint_THTPad_2.0x2.0mm_Drill1.0mm, symbol Connector:TestPoint
Connections:
- net +12V: now also J_POWER201.10 (Pin_10), J_POWER201.9 (Pin_9), TP235.1
- net -12V: now also J_POWER201.1 (Pin_1), J_POWER201.2 (Pin_2), TP236.1
- net -5V: now also TP237.1
- net GND: now also J_POWER201.3 (Pin_3), J_POWER201.4 (Pin_4), J_POWER201.5 (Pin_5), J_POWER201.6 (Pin_6), J_POWER201.7 (Pin_7), J_POWER201.8 (Pin_8)

Commit message: Updated and checked Core board BOM
ref https://github.com/shmoergh/hog/issues/19
Parts:
- C201, C202: LCSC C134220 -> C2836437; Vendor (none) -> JLCPCB
- C201, C202: LCSC C110229 -> C3344; Vendor (none) -> JLCPCB
- C203, C204, R217, R220, U202, U223: Vendor (none) -> JLCPCB
- J_POWER201: Part No. (none) -> 737-RS2-10-G; Part URL (none) -> https://mou.sr/3ZuUKrQ; Vendor (none) -> Mouser; now in the parts list

Commit message: Added JLCPCB production files to Core
ref https://github.com/shmoergh/hog/issues/19
Parts:
- C201, C202: FT Rotation Offset (none) -> 180
Changed lines of the file:
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@@
+			)
+		)
+		(property "FT Rotation Offset" "180"
+			(at 30.48 173.99 0)
+			(effects
+				(font
+					(size 1.27 1.27)
+				)
+				(hide yes)
 			)
 		)
@@
 			)
 		)
+		(property "FT Rotation Offset" "180"
+			(at 76.2 173.99 0)
+			(effects
+				(font
+					(size 1.27 1.27)
+				)
+				(hide yes)
+			)
+		)
 		(pin "1"
 		)
@@
 			)
 		)
+		(property "FT Rotation Offset" "180"
+			(at 45.72 181.61 0)
+			(effects
+				(font
+					(size 1.27 1.27)
+				)
+				(hide yes)
+			)
+		)
 		(pin "1"
 		)
@@
 			)
 		)
+		(property "FT Rotation Offset" "180"
+			(at 30.48 181.61 0)
+			(effects
+				(font
+					(size 1.27 1.27)
+				)
+				(hide yes)
+			)
+		)
 		(pin "1"
 		)
@@
 			)
 		)
+		(property "FT Rotation Offset" "180"
+			(at 45.72 173.99 0)
+			(effects
+				(font
+					(size 1.27 1.27)
+				)
+				(hide yes)
+			)
+		)
 		(pin "1"
 		)
@@
 			(at 76.2 181.61 0)
 			(effects
+				(font
+					(size 1.27 1.27)
+				)
+				(hide yes)
+			)
+		)
+		(property "FT Rotation Offset" "180"
+			(at 76.2 181.61 0)
+			(effects
